File: Deliverable10PCB/FinalPCB.kicad_sch (KiCad schematic)
At the start: 61 parts, among them J2 PiHeaderM, Q1 NMOS, Q2 PMOS, U1 MCP4131-xxxx-P, U10 MCP4131-xxxx-P, U11 MCP4131-xxxx-P, U12 LM741, U13 MCP4131-xxxx-P, U14 TL081, U2 LM741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

Commit message: changed steps at pos
Parts:
- removed U10, U11: MCP4131-xxxx-P, Package_DIP:DIP-8_W7.62mm, symbol Potentiometer_Digital:MCP4131-xxxx-P
- added C4, C5: 10nf, Capacitor_SMD:CP_Elec_3x5.3, symbol Device:C
- added R30, R35: 220k, Resistor_SMD:R_0201_0603Metric, symbol Device:R
- added R31, R32, R33, R34: 100k, Resistor_SMD:R_0201_0603Metric, symbol Device:R
- added U10, U11: TL081, Package_DIP:DIP-8_W7.62mm, symbol Amplifier_Operational:TL081
- added U15: MCP4231-103E_P, Package_DIP:DIP-8_W7.62mm, symbol MCP4231:MCP4231-103E_P
- U14: footprint (none) -> Package_DIP:DIP-8_W7.62mm
Connections:
- net +12V: now also U10.7 (V+), U11.7 (V+)
- net +3.3V: no longer 10k3.1, 10k4.1
- net -12V: now also U10.4 (V-), U11.4 (V-)
- net GND: now also R31.2, R34.2, U15.10 (P0B), U15.4 (VSS), U15.5 (P1B); no longer J2.14, J2.20, J2.25, J2.30, J2.34, J2.39, J2.6, J2.9, U5.4 (V_{SS})
- net GPIO10*: now also U1.3 (SDI/SDO), U15.3 (SDI); no longer J2.23, U13.2 (SCK), U5.2 (SCK)
- net GPIO13*: now also C3.2, U13.6 (P0W); no longer U13.5 (P0A)
- net GPIO18*: no longer 10k4.2, U4.2
- net GPIO23*: no longer 10k3.2, U4.1
- net GPIO9*: now also U15.13 (SDO)
- net CE1: now reaches U1.1 (~{CS})
- net CE1: now also J2.26, U5.1 (~{CS})
- net GPIO11*: now reaches U1.2 (SCK)
- net GPIO11*: now also J2.23, U13.2 (SCK), U5.2 (SCK), U15.2 (SCK)
- net at R22.1, R22.2, R24.1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: now also U15.6 (P1W)
- net at R29.2, U14.6: now also R32.2
- net at U9.3 (+): now also U15.9 (P0W)
- net 3V3GPIO* renamed 3.3V
- net 3.3V: now also 10k3.1, 10k4.1, U13.5 (P0A), U15.14 (VDD), U15.7 (P1A), U15.8 (P0A); no longer U5.5 (P0A), U5.8 (V_{DD})
- net 5VGPIO* renamed 5V
- net GPIO7* renamed CE0
- net CE0: now also J2.24, U15.1 (~CS); no longer J2.26
- removed net GPIO8*: J2.24, U5.1 (~{CS})
- new net: 10k3.2, U4.1
- new net: C4.2, R30.1, R32.1, U10.2 (-)
- new net: C4.1, R30.2, R33.2, U10.6
- new net: 10k4.2, U4.2
- new net: C5.2, R33.1, R35.1, U11.2 (-)
- new net: C5.1, R35.2, U11.6
- new net: R31.1, U10.3 (+)
- new net: R34.1, U11.3 (+)
- new net: U5.5 (P0A), U5.8 (V_{DD})
- new net GND*GPIO: J2.14, J2.20, J2.25, J2.30, J2.34, J2.39, J2.6, J2.9
Other:
- note added: "Square Wave/Sine Generator"
- note removed: "Square Wave Generator"
- moved on the sheet: C1, C2, C3, D1, D3, J2, Q1, Q2, R1, R10, R11, R12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
