File: Deliverable8PCB/FinalPCB.kicad_pcb (KiCad board)
At the start: 2 copper layers, 61 parts, among them J2 PiHeaderM, Q1 NMOS, Q2 PMOS, U1 MCP4131-xxxx-P, U10 MCP4131-xxxx-P, U11 MCP4131-xxxx-P, U12 LM741, U13 MCP4131-xxxx-P, U14 TL081, U2 LM741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

Commit message: changed steps at pos
Parts:
- added C4: 10nf, Capacitor_SMD:CP_Elec_3x5.3, F.Cu at (125.2, 42.8)
- added C5: 10nf, Capacitor_SMD:CP_Elec_3x5.3, F.Cu at (125.2, 29.5)
- added R30: 220k, Resistor_SMD:R_0201_0603Metric, F.Cu at (114.9, 70.8)
- added R31: 100k, Resistor_SMD:R_0201_0603Metric, F.Cu at (101.2, 81.2)
- added R32: 100k, Resistor_SMD:R_0201_0603Metric, F.Cu at (100.8, 76.5)
- added R33: 100k, Resistor_SMD:R_0201_0603Metric, F.Cu at (126.4, 55.5)
- added R34: 100k, Resistor_SMD:R_0201_0603Metric, F.Cu at (63.6, 46.5)
- added R35: 220k, Resistor_SMD:R_0201_0603Metric, F.Cu at (128.1, 60.5)
- added U15: MCP4231-103E_P, Package_DIP:DIP-8_W7.62mm, F.Cu at (51.1, 30.5)
- U10, U11: value MCP4131-xxxx-P -> TL081
- moved U10 69.5 mm to (107.9, 74.7)
- moved C3 53.6 mm to (111.8, 30.0)
- moved C1 22.2 mm to (125.2, 36.5)
- moved C2 19.7 mm to (125.0, 49.2)
- moved R27 16.1 mm to (93.8, 70.2)
- moved U13 13.8 mm to (114.3, 46.7), turned to -90 degrees
- moved U4 12.1 mm to (110.8, 38.8), turned to 90 degrees
- moved R28 8.73 mm to (102.8, 70.8)
- moved R29 6.90 mm to (98.9, 71.2)
- moved U11 3.74 mm to (52.2, 43.9)
Connections:
- net /5VGPIO* renamed /5V
- 10k3 pad 1: +3.3V -> /3.3V
- 10k3 pad 2: /GPIO23* -> Net-(10k3-Pad2)
- 10k4 pad 1: +3.3V -> /3.3V
- 10k4 pad 2: /GPIO18* -> Net-(10k4-Pad2)
- C3 pad 2: Net-(U13-P0W) -> /GPIO13*
- J2 pad 1: /3V3GPIO* -> /3.3V
- J2 pad 14: GND -> /GND*GPIO
- J2 pad 17: /3V3GPIO* -> /3.3V
- J2 pad 20: GND -> /GND*GPIO
- J2 pad 23: /GPIO10* -> /GPIO11*
- J2 pad 24: /GPIO8* -> /CE0
- J2 pad 25: GND -> /GND*GPIO
- J2 pad 26: /GPIO7* -> /CE1
- J2 pad 30: GND -> /GND*GPIO
- J2 pad 34: GND -> /GND*GPIO
- J2 pad 39: GND -> /GND*GPIO
- J2 pad 6: GND -> /GND*GPIO
- J2 pad 9: GND -> /GND*GPIO
- R22 pad 1: Net-(U10-P0W) -> Net-(U15-P1W)
- R22 pad 2: Net-(U10-P0W) -> Net-(U15-P1W)
- R24 pad 1: Net-(U10-P0W) -> Net-(U15-P1W)
- U1 pad 1: unconnected-(U1-~{CS}-Pad1) -> /CE1
- U1 pad 2: unconnected-(U1-SCK-Pad2) -> /GPIO11*
- U1 pad 3: unconnected-(U1-SDI/SDO-Pad3) -> /GPIO10*
- U10 pad 1: /GPIO7* -> unconnected-(U10-NULL-Pad1)
- U10 pad 2: /GPIO10* -> Net-(U10--)
- U10 pad 3: /GPIO10* -> Net-(U10-+)
- U10 pad 4: GND -> -12V
- U10 pad 5: /3V3GPIO* -> unconnected-(U10-NULL-Pad5)
- U10 pad 6: Net-(U10-P0W) -> Net-(C4-Pad1)
- U10 pad 7: GND -> +12V
- U10 pad 8: /3V3GPIO* -> unconnected-(U10-NC-Pad8)
- U11 pad 1: /GPIO7* -> unconnected-(U11-NULL-Pad1)
- U11 pad 2: /GPIO10* -> Net-(U11--)
- U11 pad 3: /GPIO10* -> Net-(U11-+)
- U11 pad 4: GND -> -12V
- U11 pad 5: /3V3GPIO* -> unconnected-(U11-NULL-Pad5)
- U11 pad 6: Net-(U11-P0W) -> Net-(C5-Pad1)
- U11 pad 7: GND -> +12V
- U11 pad 8: /3V3GPIO* -> unconnected-(U11-NC-Pad8)
- U13 pad 1: /GPIO7* -> /CE0
- U13 pad 2: /GPIO10* -> /GPIO11*
- U13 pad 5: /GPIO13* -> /3.3V
- U13 pad 6: Net-(U13-P0W) -> /GPIO13*
- U13 pad 8: /3V3GPIO* -> /3.3V
- U4 pad 1: /GPIO23* -> Net-(10k3-Pad2)
- U4 pad 2: /GPIO18* -> Net-(10k4-Pad2)
- U5 pad 1: /GPIO8* -> /CE1
- U5 pad 2: /GPIO10* -> /GPIO11*
- U5 pad 4: GND -> unconnected-(U5-V_{SS}-Pad4)
- U5 pad 5: /3V3GPIO* -> Net-(U5-P0A)
- U5 pad 8: /3V3GPIO* -> Net-(U5-P0A)
- U7 pad 2: Net-(U10-P0W) -> Net-(U15-P1W)
- U9 pad 3: Net-(U11-P0W) -> Net-(U15-P0W)
Routing:
- net /3.3V: track 0.00 -> 185.2 mm
- net /3V3GPIO*: track 156.4 -> 0.00 mm
- net (no net): track 0.00 -> 131.1 mm, vias 0 -> 2
- net /GPIO7*: track 113.7 -> 0.00 mm, vias 2 -> 0
- net Net-(U15-P1W): track 0.00 -> 80.8 mm, vias 0 -> 3
- net Net-(U10-P0W): track 80.8 -> 0.00 mm, vias 3 -> 0
- net /GPIO10*: track 133.7 -> 64.4 mm
- net Net-(U13-P0W): track 64.2 -> 0.00 mm, vias 1 -> 0
- net /GPIO13*: track 141.2 -> 205.4 mm, vias 1 -> 2
- net Net-(U5-P0A): track 0.00 -> 50.2 mm
- net Net-(C3-Pad1): track 21.9 -> 0.00 mm, vias 2 -> 0
- net -12V: track 232.8 -> 254.7 mm, vias 2 -> 4
- net /GPIO8*: track 17.4 -> 0.00 mm
- net Net-(C4-Pad1): track 0.00 -> 14.0 mm
- net GND: track 359.8 -> 350.1 mm
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